File: RGB_LEDS/RGB_LEDS.kicad_pcb (KiCad board)
At the start: 2 copper layers, 21.7 x 31.4 mm, 22 parts, among them IC2 INA180A4IDBVR, J2 22122021, SW1 TSC015A05026A, U1 MY-2032-08, U3 STM32C011F6U6TR, U5 TPS613221ADBV

Commit message: selector
Routing:
- net +3.3V: track 63.0 -> 63.5 mm
Changed lines of the file:
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@@
   (segment (start 160.558 91.419) (end 161.203 90.774) (width 0.25) (layer "B.Cu") (net 6))
   (segment (start 161.203 90.774) (end 162.849 90.774) (width 0.25) (layer "B.Cu") (net 6))
-  (segment (start 153.319 85.824826) (end 153.319 87.313) (width 0.3) (layer "F.Cu") (net 7))
   (segment (start 154.60472 84.539106) (end 154.60472 76.33208) (width 0.3) (layer "F.Cu") (net 7))
+  (segment (start 154.520066 86.986) (end 154.193066 87.313) (width 0.3) (layer "F.Cu") (net 7))
   (segment (start 166.409 94.231024) (end 166.409 97.609) (width 0.3) (layer "F.Cu") (net 7))
   (segment (start 147.664999 99.776) (end 148.564999 100.676) (width 0.3) (layer "F.Cu") (net 7))
@@
   (segment (start 147.354 99.775) (end 147.355 99.776) (width 0.3) (layer "F.Cu") (net 7))
   (segment (start 160.725 89.286) (end 156.046025 89.286) (width 0.3) (layer "F.Cu") (net 7))
-  (segment (start 154.520066 84.62376) (end 153.319 85.824826) (width 0.3) (layer "F.Cu") (net 7))
   (segment (start 166.203976 94.026) (end 166.409 94.231024) (width 0.3) (layer "F.Cu") (net 7))
   (segment (start 154.520066 87.760041) (end 154.520066 84.62376) (width 0.3) (layer "F.Cu") (net 7))
@@
   (segment (start 161.412 98.6405) (end 161.412 90.459) (width 0.3) (layer "F.Cu") (net 7))
   (segment (start 161.433 88.578) (end 160.725 89.286) (width 0.3) (layer "F.Cu") (net 7))
+  (segment (start 154.193066 87.313) (end 153.319 87.313) (width 0.3) (layer "F.Cu") (net 7))
   (segment (start 165.709 94.026) (end 166.203976 94.026) (width 0.3) (layer "F.Cu") (net 7))
   (segment (start 163.4475 100.5705) (end 163.4475 100.676) (width 0.3) (layer "F.Cu") (net 7))
@@
   (segment (start 156.046025 89.286) (end 154.520066 87.760041) (width 0.3) (layer "F.Cu") (net 7))
   (segment (start 161.426 88.585) (end 161.433 88.578) (width 0.3) (layer "F.Cu") (net 7))
+  (segment (start 154.520066 84.62376) (end 154.520066 86.986) (width 0.3) (layer "F.Cu") (net 7))
   (segment (start 146.241 98.2825) (end 146.241 99.761) (width 0.3) (layer "F.Cu") (net 7))
   (segment (start 147.355 99.776) (end 147.664999 99.776) (width 0.3) (layer "F.Cu") (net 7))
